File: schematics/kicad/ina326 theoretical schematic.kicad_sch (KiCad schematic)
At the start: 60 parts, among them IC1 OH49E, IC2 OH49E, IC3 OH49E, IC4 OH49E, IC5 REF1933AIDDCT, IC6 OH49E, IC7 TEENSY_4.0, J1 Conn_COILS1_male, J2 Conn_COILS2_male, J3 Jack-12V DC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

Commit message: Add files via upload
Parts:
- added C10: 0.5 nF, symbol Device:C_Small
- added R5: 200k, symbol Device:R
- renumbered C10 to C11, C11 to C12, C12 to C13, C13 to C14, C14 to C15, R9 to R10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
Connections:
- net VDD: now also C10.2, R5.2
- net at U7.5 (R2): now also C10.1, R5.1
